File: _autosave-gauss_meter_kicad.kicad_pcb (KiCad board)
At the start: 2 copper layers, 110 x 105 mm, 23 parts, among them SW3_HDR1 1985823, U1 LM258P, U2 LM358N_NOPB, U3 ESP32-DEVKITC-32D

Commit message: finalized layout, generate gerber
Parts:
- added ?: , , F.Cu at (73.4, 37.8)
- added ?: , , F.Cu at (74.7, 149.6)
- added ?: , , F.Cu at (186.4, 149.9)
- added ?: , , F.Cu at (184.6, 92.1)
- added ?: , , F.Cu at (72.3, 91.3)
- added ?: , , F.Cu at (184.4, 36.8)
Other:
- board size 110 x 105 mm -> 120 x 120 mm
- board text added: "© Soham Chakraborty Mukut Debnath Panthadip Maji ISD Lab - Group 1, 2024"
Changed lines of the file:
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@@
       (outputformat 1)
       (mirror false)
-      (drillshape 1)
+      (drillshape 0)
       (scaleselection 1)
-      (outputdirectory "")
+      (outputdirectory "CAM/")
     )
   )
@@
   (net 56 "unconnected-(U4-A2-Pad9)")
   (net 57 "unconnected-(U4-A3-Pad10)")
+  (footprint "" (layer "F.Cu")
+    (at 73.406 37.846)
+    (fp_text reference "" (at 0 0) (layer "F.SilkS")
+        (effects (font (size 1.27 1.27) (thickness 0.15)))
+    )
+    (fp_text value "" (at 0 0) (layer "F.SilkS")
+        (effects (font (size 1.27 1.27) (thickness 0.15)))
+    )
+    (pad "" np_thru_hole circle (at 1.594 1.154) (size 4 4) (drill 4) (layers "F&B.Cu" "*.Mask"))
+  )
   (footprint "1985823:PHOENIX_1985823" (layer "F.Cu")
     (at 90.16 96.698 90)
@@
     (pad "2" thru_hole circle (at 5.71 -3.6 90) (size 1.65 1.65) (drill 1.1) (layers "*.Cu" "*.Mask")
       (net 18 "/SW3") (pinfunction "2") (pintype "passive") (solder_mask_margin 0.102))
+  )
+  (footprint "" (layer "F.Cu")
+    (at 74.676 149.606)
+    (fp_text reference "" (at 0 0) (layer "F.SilkS")
+        (effects (font (size 1.27 1.27) (thickness 0.15)))
+    )
+    (fp_text value "" (at 0 0) (layer "F.SilkS")
+        (effects (font (size 1.27 1.27) (thickness 0.15)))
+    )
+    (pad "" np_thru_hole circle (at 0.324 -0.606) (size 4 4) (drill 4) (layers "F&B.Cu" "*.Mask"))
   )
   (footprint "R_gauss_custom:R_gauss_custom" (layer "F.Cu")
@@
       (net 23 "/+12V") (pinfunction "VCC") (pintype "power_in") (solder_mask_margin 0.102))
   )
+  (footprint "" (layer "F.Cu")
+    (at 186.436 149.86)
+    (fp_text reference "" (at 0 0) (layer "F.SilkS")
+        (effects (font (size 1.27 1.27) (thickness 0.15)))
+    )
+    (fp_text value "" (at 0 0) (layer "F.SilkS")
+        (effects (font (size 1.27 1.27) (thickness 0.15)))
+    )
+    (pad "" np_thru_hole circle (at -1.436 -0.86) (size 4 4) (drill 4) (layers "F&B.Cu" "*.Mask"))
+  )
   (footprint "R_gauss_custom:R_gauss_custom" (layer "F.Cu")
     (at 103.822 70.612)
@@
       (rotate (xyz 0 0 0))
     )
+  )
+  (footprint "" (layer "F.Cu")
+    (at 184.588 92.064)
+    (fp_text reference "" (at 0 0) (layer "F.SilkS")
+        (effects (font (size 1.27 1.27) (thickness 0.15)))
+    )
+    (fp_text value "" (at 0 0) (layer "F.SilkS")
+        (effects (font (size 1.27 1.27) (thickness 0.15)))
+    )
+    (pad "" np_thru_hole circle (at 0.412 1.936) (size 4 4) (drill 4) (layers "F&B.Cu" "*.Mask"))
   )
   (footprint "R_gauss_custom:R_gauss_custom" (layer "F.Cu")
@@
       (net 3 "GND") (pinfunction "03") (pintype "passive") (solder_mask_margin 0.102))
   )
+  (footprint "" (layer "F.Cu")
+    (at 72.32 91.302)
+    (fp_text reference "" (at 0 0) (layer "F.SilkS")
+        (effects (font (size 1.27 1.27) (thickness 0.15)))
+    )
+    (fp_text value "" (at 0 0) (layer "F.SilkS")
+        (effects (font (size 1.27 1.27) (thickness 0.15)))
+    )
+    (pad "" np_thru_hole circle (at 2.68 2.698) (size 4 4) (drill 4) (layers "F&B.Cu" "*.Mask"))
+  )
   (footprint "R_gauss_custom:R_gauss_custom" (layer "F.Cu")
     (at 150 87 -90)
@@
       (rotate (xyz 0 0 0))
     )
+  )
+  (footprint "" (layer "F.Cu")
+    (at 184.404 36.83)
+    (fp_text reference "" (at 0 0) (layer "F.SilkS")
+        (effects (font (size 1.27 1.27) (thickness 0.15)))
+    )
+    (fp_text value "" (at 0 0) (layer "F.SilkS")
+        (effects (font (size 1.27 1.27) (thickness 0.15)))
+    )
+    (pad "" np_thru_hole circle (at 0.596 2.17) (size 4 4) (drill 4) (layers "F&B.Cu" "*.Mask"))
   )
   (footprint "ads1115_custom:ads1115" (layer "B.Cu")
@@
   (gr_rect (start 92.094 46.294) (end 142.094 66.294)
     (stroke (width 0.15) (type default)) (fill none) (layer "F.SilkS"))
-  (gr_rect (start 75 42.5) (end 185 147.5)
+  (gr_rect (start 70 34) (end 190 154)
     (stroke (width 0.1) (type default)) (fill none) (layer "Edge.Cuts"))
+  (gr_text "© Soham Chakraborty \n   Mukut Debnath\n   Panthadip Maji \nISD Lab - Group 1, 2024" (at 99.568 44.45) (layer "F.SilkS")
+    (effects (font (size 1.5 1.5) (thickness 0.3) bold) (justify left bottom))
+  )
   (segment (start 114.352 114.808) (end 113.35 115.81) (width 0.25) (layer "F.Cu") (net 1))
   (segment (start 155.5949 110.0891) (end 150.876 114.808) (width 0.25) (layer "F.Cu") (net 1))
@@
     (connect_pads (clearance 0.54))
     (min_thickness 0.25) (filled_areas_thickness no)
-    (fill (thermal_gap 0.5) (thermal_bridge_width 0.5))
+    (fill yes (thermal_gap 0.5) (thermal_bridge_width 0.5))
     (polygon
       (pts
@@
     (connect_pads (clearance 0.5))
     (min_thickness 0.25) (filled_areas_thickness no)
-    (fill (thermal_gap 0.5) (thermal_bridge_width 0.5))
+    (fill yes (thermal_gap 0.5) (thermal_bridge_width 0.5))
     (polygon
       (pts
